Commit message: update urdf

File: assets/urdf/g1_description/g1_29dof_with_left_linkerhand.urdf (robot description, URDF)
Before this commit: robot g1_29dof, 62 links, 61 joints
Joints:
- joint left_ankle_pitch_joint: axis 0 1 0 -> (none); limit lower=-0.87267 upper=0.5236 effort=35 velocity=30 -> (none); type revolute -> fixed
- joint left_ankle_roll_joint: axis 1 0 0 -> (none); limit lower=-0.2618 upper=0.2618 effort=35 velocity=30 -> (none); type revolute -> fixed
- joint left_hip_pitch_joint: axis 0 1 0 -> (none); limit lower=-2.5307 upper=2.8798 effort=88 velocity=32 -> (none); type revolute -> fixed
- joint left_hip_roll_joint: axis 1 0 0 -> (none); limit lower=-0.5236 upper=2.9671 effort=88 velocity=32 -> (none); type revolute -> fixed
- joint left_hip_yaw_joint: axis 0 0 1 -> (none); limit lower=-2.7576 upper=2.7576 effort=88 velocity=32 -> (none); type revolute -> fixed
- joint left_knee_joint: axis 0 1 0 -> (none); limit lower=-0.087267 upper=2.8798 effort=139 velocity=20 -> (none); type revolute -> fixed
- joint rh_index_dip: axis 0 1 0 -> (none); limit lower=0 upper=1.43 effort=100 velocity=1 -> (none); mimic joint=rh_index_mcp_pitch multiplier=0.89 offset=0 -> (none); type revolute -> fixed
- joint rh_index_mcp_pitch: axis 0 1 0 -> (none); limit lower=0 upper=1.60 effort=100 velocity=1 -> (none); type revolute -> fixed
- joint rh_middle_dip: axis 0 1 0 -> (none); limit lower=0 upper=1.43 effort=100 velocity=1 -> (none); mimic joint=rh_middle_mcp_pitch multiplier=0.89 offset=0 -> (none); type revolute -> fixed
- joint rh_middle_mcp_pitch: axis 0 1 0 -> (none); limit lower=0 upper=1.60 effort=100 velocity=1 -> (none); type revolute -> fixed
- joint rh_pinky_dip: axis 0 1 0 -> (none); limit lower=0 upper=1.43 effort=100 velocity=1 -> (none); mimic joint=rh_pinky_mcp_pitch multiplier=0.89 offset=0 -> (none); type revolute -> fixed
- joint rh_pinky_mcp_pitch: axis 0 1 0 -> (none); limit lower=0 upper=1.60 effort=100 velocity=1 -> (none); type revolute -> fixed
- joint rh_ring_dip: axis 0 1 0 -> (none); limit lower=0 upper=1.43 effort=100 velocity=1 -> (none); mimic joint=rh_ring_mcp_pitch multiplier=0.89 offset=0 -> (none); type revolute -> fixed
- joint rh_ring_mcp_pitch: axis 0 1 0 -> (none); limit lower=0 upper=1.60 effort=100 velocity=1 -> (none); type revolute -> fixed
- joint rh_thumb_cmc_pitch: axis 0 1 0 -> (none); limit lower=0 upper=0.58 effort=100 velocity=1 -> (none); type revolute -> fixed
- joint rh_thumb_cmc_yaw: axis 0 0 -1 -> (none); limit lower=0 upper=1.36 effort=100 velocity=1 -> (none); type revolute -> fixed
- joint rh_thumb_ip: axis 0 1 0 -> (none); limit lower=0 upper=1.08 effort=100 velocity=1 -> (none); mimic joint=rh_thumb_cmc_pitch multiplier=1.86 offset=0 -> (none); type revolute -> fixed
- joint right_ankle_pitch_joint: axis 0 1 0 -> (none); limit lower=-0.87267 upper=0.5236 effort=35 velocity=30 -> (none); type revolute -> fixed
- joint right_ankle_roll_joint: axis 1 0 0 -> (none); limit lower=-0.2618 upper=0.2618 effort=35 velocity=30 -> (none); type revolute -> fixed
- joint right_elbow_joint: axis 0 1 0 -> (none); limit lower=-1.0472 upper=2.0944 effort=25 velocity=37 -> (none); type revolute -> fixed
- joint right_hip_pitch_joint: axis 0 1 0 -> (none); limit lower=-2.5307 upper=2.8798 effort=88 velocity=32 -> (none); type revolute -> fixed
- joint right_hip_roll_joint: axis 1 0 0 -> (none); limit lower=-2.9671 upper=0.5236 effort=88 velocity=32 -> (none); type revolute -> fixed
- joint right_hip_yaw_joint: axis 0 0 1 -> (none); limit lower=-2.7576 upper=2.7576 effort=88 velocity=32 -> (none); type revolute -> fixed
- joint right_knee_joint: axis 0 1 0 -> (none); limit lower=-0.087267 upper=2.8798 effort=139 velocity=20 -> (none); type revolute -> fixed
- joint right_shoulder_pitch_joint: axis 0 1 0 -> (none); limit lower=-3.0892 upper=2.6704 effort=25 velocity=37 -> (none); type revolute -> fixed
- joint right_shoulder_roll_joint: axis 1 0 0 -> (none); limit lower=-2.2515 upper=1.5882 effort=25 velocity=37 -> (none); type revolute -> fixed
- joint right_shoulder_yaw_joint: axis 0 0 1 -> (none); limit lower=-2.618 upper=2.618 effort=25 velocity=37 -> (none); type revolute -> fixed
- joint right_wrist_pitch_joint: axis 0 1 0 -> (none); limit lower=-1.614429558 upper=1.614429558 effort=5 velocity=22 -> (none); type revolute -> fixed
- joint right_wrist_roll_joint: axis 1 0 0 -> (none); limit lower=-1.972222054 upper=1.972222054 effort=25 velocity=37 -> (none); type revolute -> fixed
- joint right_wrist_yaw_joint: axis 0 0 1 -> (none); limit lower=-1.614429558 upper=1.614429558 effort=5 velocity=22 -> (none); type revolute -> fixed
- joint waist_pitch_joint: axis 0 1 0 -> (none); limit lower=-0.52 upper=0.52 effort=35 velocity=30 -> (none); type revolute -> fixed
- joint waist_roll_joint: axis 1 0 0 -> (none); limit lower=-0.52 upper=0.52 effort=35 velocity=30 -> (none); type revolute -> fixed
- joint waist_yaw_joint: axis 0 0 1 -> (none); limit lower=-2.618 upper=2.618 effort=88 velocity=32 -> (none); type revolute -> fixed
