Commit message: add mimic joint control but with some bugs

File: assets/urdf/g1_description/g1_29dof_with_left_sharpa_correct.urdf (robot description, URDF)
Before this commit: robot g1_29dof, 62 links, 61 joints
Links:
- removed link lh_hand_base_link
- removed link lh_index_distal
- removed link lh_index_proximal
- removed link lh_middle_distal
- removed link lh_middle_proximal
- removed link lh_pinky_distal
- removed link lh_pinky_proximal
- removed link lh_ring_distal
- removed link lh_ring_proximal
- removed link lh_thumb_distal
- removed link lh_thumb_metacarpals
- removed link lh_thumb_metacarpals_base2
- removed link rh_hand_base_link
- removed link rh_index_distal
- removed link rh_index_proximal
- removed link rh_middle_distal
- removed link rh_middle_proximal
- removed link rh_pinky_distal
- removed link rh_pinky_proximal
- removed link rh_ring_distal
- removed link rh_ring_proximal
- removed link rh_thumb_distal
- removed link rh_thumb_metacarpals
- removed link rh_thumb_metacarpals_base2
- added link left_hand_C_MC, mass 0.72045; collision mesh filename=left_sharpa_meshes/left_hand_C_MC.STL; visual mesh filename=left_sharpa_meshes/left_hand_C_MC_visual.STL
- added link left_index_DP, mass 0.003002; collision mesh filename=left_sharpa_meshes/left_DP.STL; visual mesh filename=left_sharpa_meshes/left_DP_visual.STL
- added link left_index_MCP_VL, mass 1.0E-06; collision mesh filename=left_sharpa_meshes/MCP_VL.STL; visual mesh filename=left_sharpa_meshes/left_MCP_VL_visual.STL
- added link left_index_MP, mass 0.02509; collision mesh filename=left_sharpa_meshes/left_MP.STL; visual mesh filename=left_sharpa_meshes/left_MP_visual.STL
- added link left_index_PP, mass 0.04138; collision mesh filename=left_sharpa_meshes/left_PP.STL; visual mesh filename=left_sharpa_meshes/left_PP_visual.STL
- added link left_index_elastomer, mass 0.00110; collision mesh filename=left_sharpa_meshes/elastomer.STL; visual mesh filename=left_sharpa_meshes/elastomer_surface.STL
- added link left_index_fingertip, mass 1.0E-06
- added link left_middle_DP, mass 0.003002; collision mesh filename=left_sharpa_meshes/left_DP.STL; visual mesh filename=left_sharpa_meshes/left_DP_visual.STL
- added link left_middle_MCP_VL, mass 1.0E-06; collision mesh filename=left_sharpa_meshes/MCP_VL.STL; visual mesh filename=left_sharpa_meshes/left_MCP_VL_visual.STL
- added link left_middle_MP, mass 0.02509; collision mesh filename=left_sharpa_meshes/left_MP.STL; visual mesh filename=left_sharpa_meshes/left_MP_visual.STL
- added link left_middle_PP, mass 0.04138; collision mesh filename=left_sharpa_meshes/left_PP.STL; visual mesh filename=left_sharpa_meshes/left_PP_visual.STL
- added link left_middle_elastomer, mass 0.00110; collision mesh filename=left_sharpa_meshes/elastomer.STL; visual mesh filename=left_sharpa_meshes/elastomer_surface.STL
- added link left_middle_fingertip, mass 1.0E-06
- added link left_pinky_DP, mass 0.003002; collision mesh filename=left_sharpa_meshes/left_DP.STL; visual mesh filename=left_sharpa_meshes/left_DP_visual.STL
- added link left_pinky_MC, mass 0.12541; collision mesh filename=left_sharpa_meshes/left_pinky_MC.STL; visual mesh filename=left_sharpa_meshes/left_pinky_MC_visual.STL
- added link left_pinky_MCP_VL, mass 1.0E-06; collision mesh filename=left_sharpa_meshes/MCP_VL.STL; visual mesh filename=left_sharpa_meshes/left_MCP_VL_visual.STL
- added link left_pinky_MP, mass 0.02509; collision mesh filename=left_sharpa_meshes/left_MP.STL; visual mesh filename=left_sharpa_meshes/left_MP_visual.STL
- added link left_pinky_PP, mass 0.04138; collision mesh filename=left_sharpa_meshes/left_PP.STL; visual mesh filename=left_sharpa_meshes/left_PP_visual.STL
- added link left_pinky_elastomer, mass 0.00110; collision mesh filename=left_sharpa_meshes/elastomer.STL; visual mesh filename=left_sharpa_meshes/elastomer_surface.STL
- added link left_pinky_fingertip, mass 1.0E-06
- added link left_ring_DP, mass 0.003002; collision mesh filename=left_sharpa_meshes/left_DP.STL; visual mesh filename=left_sharpa_meshes/left_DP_visual.STL
- added link left_ring_MCP_VL, mass 1.0E-06; collision mesh filename=left_sharpa_meshes/MCP_VL.STL; visual mesh filename=left_sharpa_meshes/left_MCP_VL_visual.STL
- added link left_ring_MP, mass 0.02509; collision mesh filename=left_sharpa_meshes/left_MP.STL; visual mesh filename=left_sharpa_meshes/left_MP_visual.STL
- added link left_ring_PP, mass 0.04138; collision mesh filename=left_sharpa_meshes/left_PP.STL; visual mesh filename=left_sharpa_meshes/left_PP_visual.STL
- added link left_ring_elastomer, mass 0.00110; collision mesh filename=left_sharpa_meshes/elastomer.STL; visual mesh filename=left_sharpa_meshes/elastomer_surface.STL
- added link left_ring_fingertip, mass 1.0E-06
- added link left_thumb_CMC_VL, mass 1.0E-06; visual mesh filename=left_sharpa_meshes/left_thumb_CMC_VL.STL
- added link left_thumb_DP, mass 0.003886; collision mesh filename=left_sharpa_meshes/left_thumb_DP.STL; visual mesh filename=left_sharpa_meshes/left_thumb_DP_visual.STL
- added link left_thumb_MC, mass 0.116; collision mesh filename=left_sharpa_meshes/left_thumb_MC.STL; visual mesh filename=left_sharpa_meshes/left_thumb_MC_visual.STL
- added link left_thumb_MCP_VL, mass 1.0E-06; visual mesh filename=left_sharpa_meshes/left_thumb_MCP_VL_visual.STL
- added link left_thumb_PP, mass 0.04955; collision mesh filename=left_sharpa_meshes/left_thumb_PP.STL; visual mesh filename=left_sharpa_meshes/left_thumb_PP_visual.STL
- added link left_thumb_elastomer, mass 0.002100; collision mesh filename=left_sharpa_meshes/thumb_elastomer.STL; visual mesh filename=left_sharpa_meshes/thumb_elastomer_surface.STL
- added link left_thumb_fingertip, mass 1.0E-06
- added link sharpa_mount, mass 0.05
Joints:
- removed joint left_linkerhand_base_joint
- removed joint lh_index_dip
- removed joint lh_index_mcp_pitch
- removed joint lh_middle_dip
- removed joint lh_middle_mcp_pitch
- removed joint lh_pinky_dip
- removed joint lh_pinky_mcp_pitch
- removed joint lh_ring_dip
- removed joint lh_ring_mcp_pitch
- removed joint lh_thumb_cmc_pitch
- removed joint lh_thumb_cmc_yaw
- removed joint lh_thumb_ip
- removed joint rh_index_dip
- removed joint rh_index_mcp_pitch
- removed joint rh_middle_dip
- removed joint rh_middle_mcp_pitch
- removed joint rh_pinky_dip
- removed joint rh_pinky_mcp_pitch
- removed joint rh_ring_dip
- removed joint rh_ring_mcp_pitch
- removed joint rh_thumb_cmc_pitch
- removed joint rh_thumb_cmc_yaw
- removed joint rh_thumb_ip
- removed joint right_linkerhand_base_joint
- added joint g1_sharpa: type fixed, parent left_wrist_yaw_link, child sharpa_mount, origin xyz=0 0 0 rpy=0 0 0
- added joint left_1_thumb_CMC_FE: type revolute, parent left_hand_C_MC, child left_thumb_CMC_VL, origin xyz=0.01 -0.026 0.0212 rpy=0 0 -1.5708, axis 0 0 1, limit lower=-0.1745 upper=1.9199 effort=3.3 velocity=11.84076833
- added joint left_2_index_MCP_FE: type revolute, parent left_hand_C_MC, child left_index_MCP_VL, origin xyz=0.001 -0.0303 0.0957 rpy=0 -1.5708 -1.5708, axis 0 0 1, limit lower=-0.17453293 upper=1.5708 effort=1.864 velocity=16.07692878
- added joint left_3_middle_MCP_FE: type revolute, parent left_hand_C_MC, child left_middle_MCP_VL, origin xyz=0 -0.01 0.0987 rpy=0 -1.5708 -1.5708, axis 0 0 1, limit lower=-0.17453293 upper=1.5708 effort=1.864 velocity=16.07692878
- added joint left_4_ring_MCP_FE: type revolute, parent left_hand_C_MC, child left_ring_MCP_VL, origin xyz=0.0015 0.0103 0.0927 rpy=0 -1.5708 -1.5708, axis 0 0 1, limit lower=-0.17453293 upper=1.5708 effort=1.864 velocity=16.07692878
- added joint left_5_pinky_CMC: type revolute, parent left_hand_C_MC, child left_pinky_MC, origin xyz=0.01136 0.0263 0.0867 rpy=-3.1416 0 3.1416, axis 0 0 1, limit lower=0 upper=0.2618 effort=0.5285 velocity=35.07416159
- added joint left_index_DIP: type revolute, parent left_index_MP, child left_index_DP, origin xyz=0.0315 0 0 rpy=0 0 0, axis 0 0 1, limit lower=0 upper=1.3963 effort=0.189369 velocity=14.66594768
- added joint left_index_MCP_AA: type revolute, parent left_index_MCP_VL, child left_index_PP, origin xyz=0 0 0 rpy=1.5708 0 0, axis 0 0 1, limit lower=-0.03491 upper=0.03491 effort=1.864 velocity=16.07692878
- added joint left_index_PIP: type revolute, parent left_index_PP, child left_index_MP, origin xyz=0.047 0 0 rpy=-1.5708 0 0, axis 0 0 1, limit lower=0 upper=1.7453 effort=0.638 velocity=11.61831603
- added joint left_index_elastomer_fix_joint: type fixed, parent left_index_DP, child left_index_elastomer, origin xyz=0 0 0 rpy=1.5707963267949 -1.5707963267949 0, axis 0 0 0
- added joint left_index_fingertip_fix_joint: type fixed, parent left_index_elastomer, child left_index_fingertip, origin xyz=0 -0.0260092574262508 0 rpy=1.5707963267949 1.5707963267949 0, axis 0 0 0
- added joint left_middle_DIP: type revolute, parent left_middle_MP, child left_middle_DP, origin xyz=0.0315 0 0 rpy=0 0 0, axis 0 0 1, limit lower=0 upper=1.3963 effort=0.189369 velocity=14.66594768
- added joint left_middle_MCP_AA: type revolute, parent left_middle_MCP_VL, child left_middle_PP, origin xyz=0 0 0 rpy=1.5708 0 0, axis 0 0 1, limit lower=-0.03491 upper=0.03491 effort=1.864 velocity=16.07692878
- added joint left_middle_PIP: type revolute, parent left_middle_PP, child left_middle_MP, origin xyz=0.047 0 0 rpy=-1.5708 0 0, axis 0 0 1, limit lower=0 upper=1.7453 effort=0.638 velocity=11.61831603
- added joint left_middle_elastomer_fix_joint: type fixed, parent left_middle_DP, child left_middle_elastomer, origin xyz=0 0 0 rpy=1.5707963267949 -1.5707963267949 0, axis 0 0 0
- added joint left_middle_fingertip_fix_joint: type fixed, parent left_middle_elastomer, child left_middle_fingertip, origin xyz=0 -0.0260092574262507 0 rpy=1.5707963267949 1.5707963267949 0, axis 0 0 0
- added joint left_pinky_DIP: type revolute, parent left_pinky_MP, child left_pinky_DP, origin xyz=0.0315 0 0 rpy=0 0 0, axis 0 0 1, limit lower=0 upper=1.3963 effort=0.189369 velocity=14.66594768
- added joint left_pinky_MCP_AA: type revolute, parent left_pinky_MCP_VL, child left_pinky_PP, origin xyz=0 0 0 rpy=1.5708 0 0, axis 0 0 1, limit lower=-0.03491 upper=0.03491 effort=1.864 velocity=16.07692878
- added joint left_pinky_MCP_FE: type revolute, parent left_pinky_MC, child left_pinky_MCP_VL, origin xyz=0.00836 0.0048 0 rpy=-1.5708 1.5708 0, axis 0 0 1, limit lower=-0.17453293 upper=1.5708 effort=1.864 velocity=16.07692878
- added joint left_pinky_PIP: type revolute, parent left_pinky_PP, child left_pinky_MP, origin xyz=0.047 0 0 rpy=-1.5708 0 0, axis 0 0 1, limit lower=0 upper=1.7453 effort=0.638 velocity=11.61831603
- added joint left_pinky_elastomer_fix_joint: type fixed, parent left_pinky_DP, child left_pinky_elastomer, origin xyz=0 0 0 rpy=1.5707963267949 -1.5707963267949 0, axis 0 0 0
- added joint left_pinky_fingertip_fix_joint: type fixed, parent left_pinky_elastomer, child left_pinky_fingertip, origin xyz=0 -0.0260092574262507 0 rpy=1.5707963267949 1.5707963267949 0, axis 0 0 0
- added joint left_ring_DIP: type revolute, parent left_ring_MP, child left_ring_DP, origin xyz=0.0315 0 0 rpy=0 0 0, axis 0 0 1, limit lower=0 upper=1.3963 effort=0.189369 velocity=14.66594768
- added joint left_ring_MCP_AA: type revolute, parent left_ring_MCP_VL, child left_ring_PP, origin xyz=0 0 0 rpy=1.5708 0 0, axis 0 0 1, limit lower=-0.03491 upper=0.03491 effort=1.864 velocity=16.07692878
- added joint left_ring_PIP: type revolute, parent left_ring_PP, child left_ring_MP, origin xyz=0.047 0 0 rpy=-1.5708 0 0, axis 0 0 1, limit lower=0 upper=1.7453 effort=0.638 velocity=11.61831603
- added joint left_ring_elastomer_fix_joint: type fixed, parent left_ring_DP, child left_ring_elastomer, origin xyz=0 0 0 rpy=1.5708 -1.5708 0, axis 0 0 0
- added joint left_ring_fingertip_fix_joint: type fixed, parent left_ring_elastomer, child left_ring_fingertip, origin xyz=0 -0.0260092574262507 0 rpy=1.5707963267949 1.5707963267949 0, axis 0 0 0
- added joint left_thumb_CMC_AA: type revolute, parent left_thumb_CMC_VL, child left_thumb_MC, origin xyz=0 -0.005 0 rpy=1.5708 -0.7854 0, axis 0 0 1, limit lower=-0.3491 upper=0.1309 effort=3.3 velocity=11.84076833
- added joint left_thumb_IP: type revolute, parent left_thumb_PP, child left_thumb_DP, origin xyz=0.039 0 0 rpy=-1.5708 0 0, axis 0 0 1, limit lower=0 upper=1.7453 effort=0.638 velocity=11.61831603
- added joint left_thumb_MCP_AA: type revolute, parent left_thumb_MCP_VL, child left_thumb_PP, origin xyz=0 0 0 rpy=1.5708 0 0, axis 0 0 1, limit lower=-0.3491 upper=0.3491 effort=1.864 velocity=16.07692878
- added joint left_thumb_MCP_FE: type revolute, parent left_thumb_MC, child left_thumb_MCP_VL, origin xyz=0.065 -0.006 -0.010392 rpy=-0.5236 0 0, axis 0 0 1, limit lower=-0.5236 upper=1.3963 effort=1.864 velocity=16.07692878
- added joint left_thumb_elastomer_fix_joint: type fixed, parent left_thumb_DP, child left_thumb_elastomer, origin xyz=0 0 0 rpy=1.5707963267949 -1.5707963267949 0, axis 0 0 0
- added joint left_thumb_fingertip_fix_joint: type fixed, parent left_thumb_elastomer, child left_thumb_fingertip, origin xyz=0 -0.0276109346321216 0 rpy=1.5707963267949 1.5707963267949 0, axis 0 0 0
- added joint sharpa_mount_joint: type fixed, parent sharpa_mount, child left_hand_C_MC, origin xyz=0.0415 0.0 0 rpy=-1.5708 0 -1.5708
